File: KiCad Files/Matterhorn-64-CORE/Matterhorn-64-CORE.kicad_pcb (KiCad board)
At the start: 4 copper layers, 78 x 77.2 mm, 177 parts, among them J1 5051104091, U1 CPU-NUS, U10 MX8330, U2 RCP-NUS, U3 74LCV125, U4 PTS9128, U5 RDRAM18-NUS, U6 MX8330, U8 PIF-NUS, U9 RDRAM18-NUS, Y1 14.3181MHz, Y2 14.705882MHz

Commit message: Updates some silkscreen issues
Routing:
- net GND: vias 667 -> 671
Changed lines of the file:
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@@
 		(tags "capacitor")
 		(property "Reference" "C53"
-			(at 0 1.16 90)
+			(at -0.107836 -1.05 90)
 			(layer "B.SilkS")
 			(effects
@@
 		(tags "capacitor")
 		(property "Reference" "C56"
-			(at 0 1.16 90)
+			(at -0.107836 -1.05 90)
 			(layer "B.SilkS")
 			(effects
@@
 		(tags "capacitor")
 		(property "Reference" "C67"
-			(at 0.93 3.55 0)
+			(at 0.93 4.1 90)
 			(layer "B.SilkS")
 			(effects
@@
 		(tags "capacitor")
 		(property "Reference" "C64"
-			(at -1.17 2.55 0)
+			(at -1.17 3 90)
 			(layer "B.SilkS")
 			(effects
@@
 		(tags "capacitor")
 		(property "Reference" "C61"
-			(at -0.12 1.55 0)
+			(at -0.12 2 90)
 			(layer "B.SilkS")
 			(effects
@@
 	)
 	(via
+		(at 144.1 129.9)
+		(size 0.6)
+		(drill 0.3)
+		(layers "F.Cu" "B.Cu")
+		(free yes)
+		(net 13)
+	)
+	(via
 		(at 186.8 70.7)
 		(size 0.6)
@@
 	)
 	(via
+		(at 145.2 129.9)
+		(size 0.6)
+		(drill 0.3)
+		(layers "F.Cu" "B.Cu")
+		(free yes)
+		(net 13)
+	)
+	(via
 		(at 157.2 61.4)
 		(size 0.6)
@@
 	)
 	(via
+		(at 143.8 128.7)
+		(size 0.6)
+		(drill 0.3)
+		(layers "F.Cu" "B.Cu")
+		(free yes)
+		(net 13)
+	)
+	(via
 		(at 122 94.4)
 		(size 0.6)
@@
 	)
 	(via
+		(at 145.5 128.1)
+		(size 0.6)
+		(drill 0.3)
+		(layers "F.Cu" "B.Cu")
+		(free yes)
+		(net 13)
+	)
+	(via
 		(at 129.5 84)
 		(size 0.6)
@@
 	)
 	(zone
+		(net 57)
+		(net_name "~{NMI}")
+		(layer "F.Cu")
+		(name "$teardrop_padvia$")
+		(hatch none 0.1)
+		(priority 30000)
+		(attr
+			(teardrop
+				(type padvia)
+			)
+		)
+		(connect_pads yes
+			(clearance 0)
+		)
+		(min_thickness 0.0254)
+		(filled_areas_thickness no)
+		(fill yes
+			(thermal_gap 0.5)
+			(thermal_bridge_width 0.5)
+			(island_removal_mode 1)
+			(island_area_min 10)
+		)
+		(polygon
+			(pts
+				(xy 125.078171 99.758748) (xy 125.147934 99.784502) (xy 125.200463 99.814001) (xy 125.268757 99.881548)
+				(xy 125.309033 99.947495) (xy 125.372209 100.045521) (xy 125.420603 100.097024) (xy 125.488004 100.149441)
+				(xy 125.655633 99.900285) (xy 125.596148 99.605764) (xy 125.444131 99.64281) (xy 125.370739 99.661579)
+				(xy 125.302005 99.669978) (xy 125.221913 99.663351) (xy 125.11445 99.637041)
+			)
+		)
+	)
+	(zone
 		(net 14)
 		(net_name "+3V3")
@@
 	)
 	(zone
-		(net 57)
-		(net_name "~{NMI}")
-		(layer "F.Cu")
-		(name "$teardrop_padvia$")
-		(hatch none 0.1)
-		(priority 30000)
-		(attr
-			(teardrop
-				(type padvia)
-			)
-		)
-		(connect_pads yes
-			(clearance 0)
-		)
-		(min_thickness 0.0254)
-		(filled_areas_thickness no)
-		(fill yes
-			(thermal_gap 0.5)
-			(thermal_bridge_width 0.5)
-			(island_removal_mode 1)
-			(island_area_min 10)
-		)
-		(polygon
-			(pts
-				(xy 125.078171 99.758748) (xy 125.147934 99.784502) (xy 125.200463 99.814001) (xy 125.268757 99.881548)
-				(xy 125.309033 99.947495) (xy 125.372209 100.045521) (xy 125.420603 100.097024) (xy 125.488004 100.149441)
-				(xy 125.655633 99.900285) (xy 125.596148 99.605764) (xy 125.444131 99.64281) (xy 125.370739 99.661579)
-				(xy 125.302005 99.669978) (xy 125.221913 99.663351) (xy 125.11445 99.637041)
-			)
-		)
-	)
-	(zone
 		(net 0)
 		(net_name "")
@@
 	)
 	(zone
-		(net 22)
-		(net_name "Net-(C59-Pad2)")
+		(net 57)
+		(net_name "~{NMI}")
 		(layer "B.Cu")
-		(hatch edge 0.5)
-		(priority 1)
+		(name "$teardrop_padvia$")
+		(hatch none 0.1)
+		(priority 30000)
+		(attr
+			(teardrop
+				(type padvia)
+			)
+		)
 		(connect_pads yes
-			(clearance 0.127)
+			(clearance 0)
 		)
-		(min_thickness 0.25)
+		(min_thickness 0.0254)
 		(filled_areas_thickness no)
 		(fill yes
 			(thermal_gap 0.5)
 			(thermal_bridge_width 0.5)
+			(island_removal_mode 1)
+			(island_area_min 10)
 		)
 		(polygon
 			(pts
-				(xy 141.8 85.82) (xy 141.8 81.8) (xy 141.337154 81.8) (xy 140.053641 83.671644) (xy 140.053641 83.894178)
-				(xy 141.374308 85.82)
+				(xy 125.279389 100.365089) (xy 125.354936 100.296733) (xy 125.417944 100.255775) (xy 125.517796 100.22501)
+				(xy 125.576712 100.216312) (xy 125.713202 100.194236) (xy 125.655382 99.899293) (xy 125.360439 99.841473)
+				(xy 125.338362 99.977964) (xy 125.325882 100.056887) (xy 125.304857 100.124171) (xy 125.26339 100.192682)
+				(xy 125.189586 100.275286)
 			)
 		)
 	)
 	(zone
-		(net 14)
-		(net_name "+3V3")
+		(net 22)
+		(net_name "Net-(C59-Pad2)")
 		(layer "B.Cu")
 		(hatch edge 0.5)
-		(priority 17)
+		(priority 1)
 		(connect_pads yes
 			(clearance 0.127)
@@
 		(polygon
 			(pts
-				(xy 143.3 70.45) (xy 142.65 70.45) (xy 141.45 70) (xy 141.45 69.35) (xy 142.65 68.85) (xy 143.3 68.85)
+				(xy 141.8 85.82) (xy 141.8 81.8) (xy 141.337154 81.8) (xy 140.053641 83.671644) (xy 140.053641 83.894178)
+				(xy 141.374308 85.82)
 			)
 		)
 	)
 	(zone
-		(net 57)
-		(net_name "~{NMI}")
+		(net 14)
+		(net_name "+3V3")
 		(layer "B.Cu")
-		(name "$teardrop_padvia$")
-		(hatch none 0.1)
-		(priority 30000)
-		(attr
-			(teardrop
-				(type padvia)
-			)
-		)
+		(hatch edge 0.5)
+		(priority 17)
 		(connect_pads yes
-			(clearance 0)
+			(clearance 0.127)
 		)
-		(min_thickness 0.0254)
+		(min_thickness 0.25)
 		(filled_areas_thickness no)
 		(fill yes
 			(thermal_gap 0.5)
 			(thermal_bridge_width 0.5)
-			(island_removal_mode 1)
-			(island_area_min 10)
 		)
 		(polygon
 			(pts
-				(xy 125.279389 100.365089) (xy 125.354936 100.296733) (xy 125.417944 100.255775) (xy 125.517796 100.22501)
-				(xy 125.576712 100.216312) (xy 125.713202 100.194236) (xy 125.655382 99.899293) (xy 125.360439 99.841473)
-				(xy 125.338362 99.977964) (xy 125.325882 100.056887) (xy 125.304857 100.124171) (xy 125.26339 100.192682)
-				(xy 125.189586 100.275286)
+				(xy 143.3 70.45) (xy 142.65 70.45) (xy 141.45 70) (xy 141.45 69.35) (xy 142.65 68.85) (xy 143.3 68.85)
 			)
 		)
@@
 	)
 	(zone
-		(net 14)
-		(net_name "+3V3")
-		(layer "B.Cu")
-		(hatch edge 0.5)
-		(priority 20)
-		(connect_pads yes
-			(clearance 0.3)
-		)
-		(min_thickness 0.25)
-		(filled_areas_thickness no)
-		(fill yes
-			(thermal_gap 0.5)
-			(thermal_bridge_width 0.5)
-		)
-		(polygon
-			(pts
-				(xy 139.8 85.8) (xy 139.8 81.9) (xy 139.1 81.9) (xy 139.1 85.8)
-			)
-		)
-	)
-	(zone
 		(net 57)
 		(net_name "~{NMI}")
@@
 			)
 		)
+	)
+	(zone
+		(net 14)
+		(net_name "+3V3")
+		(layer "B.Cu")
+		(hatch edge 0.5)
+		(priority 20)
+		(connect_pads yes
+			(clearance 0.3)
+		)
+		(min_thickness 0.25)
+		(filled_areas_thickness no)
+		(fill yes
+			(thermal_gap 0.5)
+			(thermal_bridge_width 0.5)
+		)
+		(polygon
+			(pts
+				(xy 139.8 85.8) (xy 139.8 81.9) (xy 139.1 81.9) (xy 139.1 85.8)
+			)
+		)

Commit message: Fixes a little silkscreen issue (R28 placement)
Parts:
- U5, U9: value RDRAM18-NUS -> N64_U11/14_RAM
Other:
- board text added: "REV 1.3 - 28/9/2026 MSF - 001"
- board text removed: "REV 1.2 - 13/5/2026 MSF - 001"
Changed lines of the file:
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@@
 			(layer "F.SilkS")
 		)
-		(fp_circle
-			(center 14.5 14.6)
-			(end 14.5 14.3)
-			(stroke
-				(width 0.1)
-				(type default)
-			)
-			(fill yes)
-			(layer "F.SilkS")
-		)
 		(pad "1" smd roundrect
 			(at 15.75 12.675 270)
@@
 		)
 		(embedded_fonts no)
-		(model "C:/Users/Timéo/Desktop/Matterhorn 64/Matterhorn Core/3D/Nintendo-IC/qfp-160.wrl"
+		(model "C:/Users/Timéo/Desktop/Matterhorn 64/Matterhorn Core/3D/Nintendo-IC/qfp-160.step"
 			(offset
-				(xyz 12.84 -14 0)
+				(xyz 13 -14 0)
 			)
 			(scale
-				(xyz 0.394 0.394 0.4)
+				(xyz 1 1 1)
 			)
 			(rotate
-				(xyz -0 -0 -90)
+				(xyz -90 -180 90)
 			)
 		)
@@
 		)
 		(embedded_fonts no)
+		(model "${KICAD9_3DMODEL_DIR}/Crystal.3dshapes/Crystal_HC49-4H_Vertical.wrl"
+			(offset
+				(xyz -2.5 0 0)
+			)
+			(scale
+				(xyz 1 1 1)
+			)
+			(rotate
+				(xyz -0 -0 -0)
+			)
+		)
 	)
 	(footprint "Capacitor_SMD:C_0402_1005Metric"
@@
 			)
 		)
-		(property "Value" "RDRAM18-NUS"
+		(property "Value" "N64_U11/14_RAM"
 			(at 0.335 1.745 0)
 			(unlocked yes)
@@
 		)
 		(embedded_fonts no)
-		(model "C:/Users/Timéo/Desktop/Matterhorn 64/Matterhorn Core/3D/Nintendo-IC/shp-32.wrl"
+		(model "C:/Users/Timéo/Desktop/Matterhorn 64/Matterhorn Core/3D/Nintendo-IC/shp-32.step"
 			(offset
-				(xyz -12.5 5.5 0)
+				(xyz -12.45 5.5 0)
 			)
 			(scale
-				(xyz 0.393 0.3937 0.3937)
+				(xyz 1 1 1)
 			)
 			(rotate
-				(xyz -0 -0 90)
+				(xyz 90 -0 90)
 			)
 		)
@@
 		)
 		(embedded_fonts no)
+		(model "${KICAD9_3DMODEL_DIR}/Crystal.3dshapes/Crystal_HC49-4H_Vertical.wrl"
+			(offset
+				(xyz -2.5 0 0)
+			)
+			(scale
+				(xyz 1 1 1)
+			)
+			(rotate
+				(xyz -0 -0 -0)
+			)
+		)
 	)
 	(footprint "Capacitor_SMD:C_0402_1005Metric"
@@
 		(tags "resistor")
 		(property "Reference" "R28"
-			(at 0 0.9 90)
+			(at 0 -0.9 90)
 			(layer "F.SilkS")
 			(effects
@@
 			)
 		)
-		(property "Value" "RDRAM18-NUS"
+		(property "Value" "N64_U11/14_RAM"
 			(at 0.335 1.745 0)
 			(unlocked yes)
@@
 		)
 		(embedded_fonts no)
-		(model "C:/Users/Timéo/Desktop/Matterhorn 64/Matterhorn Core/3D/Nintendo-IC/shp-32.wrl"
+		(model "C:/Users/Timéo/Desktop/Matterhorn 64/Matterhorn Core/3D/Nintendo-IC/shp-32.step"
 			(offset
-				(xyz -12.5 5.5 0)
+				(xyz -12.45 5.5 0)
 			)
 			(scale
-				(xyz 0.393 0.3937 0.3937)
+				(xyz 1 1 1)
 			)
 			(rotate
-				(xyz -0 -0 90)
+				(xyz 90 -0 90)
 			)
 		)
@@
 			(layer "F.SilkS")
 		)
-		(fp_circle
-			(center 14.2 14)
-			(end 14.5 14)
-			(stroke
-				(width 0.1)
-				(type default)
-			)
-			(fill yes)
-			(layer "F.SilkS")
-		)
 		(pad "1" smd roundrect
 			(at 15.75 11.6)
@@
 		)
 		(embedded_fonts no)
-		(model "C:/Users/Timéo/Desktop/Matterhorn 64/Matterhorn Core/3D/Nintendo-IC/qfp-120_08.wrl"
+		(model "C:/Users/Timéo/Desktop/Matterhorn 64/Matterhorn Core/3D/Nintendo-IC/qfp-120_08.step"
 			(offset
 				(xyz 0 0 0)
 			)
 			(scale
-				(xyz 1 1 1)
+				(xyz 2.54 2.54 2.54)
 			)
 			(rotate
-				(xyz -0 -0 -90)
+				(xyz 90 -0 -90)
 			)
 		)
@@
 		(layer "F.SilkS")
 	)
+	(gr_circle
+		(center 180.2 94.7)
+		(end 180.2 94.4)
+		(stroke
+			(width 0.1)
+			(type default)
+		)
+		(fill yes)
+		(layer "F.SilkS")
+	)
 	(gr_line
 		(start 135.1404 114)
@@
 		(layer "F.SilkS")
 	)
+	(gr_circle
+		(center 142.8 94.1)
+		(end 142.8 93.8)
+		(stroke
+			(width 0.1)
+			(type default)
+		)
+		(fill yes)
+		(layer "F.SilkS")
+	)
 	(gr_line
 		(start 142 82.15)
@@
 		)
 	)
-	(gr_text "REV 1.2 - 13/5/2026\nMSF - 001"
+	(gr_text "REV 1.3 - 28/9/2026\nMSF - 001"
 		(at 115.5 60.575 0)
 		(layer "F.SilkS")
@@
 	)
 	(zone
-		(net 57)
-		(net_name "~{NMI}")
+		(net 14)
+		(net_name "+3V3")
 		(layer "F.Cu")
-		(name "$teardrop_padvia$")
-		(hatch none 0.1)
-		(priority 30000)
-		(attr
-			(teardrop
-				(type padvia)
-			)
-		)
+		(hatch edge 0.5)
+		(priority 10)
 		(connect_pads yes
-			(clearance 0)
+			(clearance 0.127)
 		)
-		(min_thickness 0.0254)
+		(min_thickness 0.25)
 		(filled_areas_thickness no)
 		(fill yes
 			(thermal_gap 0.5)
 			(thermal_bridge_width 0.5)
-			(island_removal_mode 1)
-			(island_area_min 10)
+			(smoothing fillet)
+			(radius 0.5)
 		)
 		(polygon
 			(pts
-				(xy 125.078171 99.758748) (xy 125.147934 99.784502) (xy 125.200463 99.814001) (xy 125.268757 99.881548)
-				(xy 125.309033 99.947495) (xy 125.372209 100.045521) (xy 125.420603 100.097024) (xy 125.488004 100.149441)
-				(xy 125.655633 99.900285) (xy 125.596148 99.605764) (xy 125.444131 99.64281) (xy 125.370739 99.661579)
-				(xy 125.302005 99.669978) (xy 125.221913 99.663351) (xy 125.11445 99.637041)
+				(xy 143.55 126.85) (xy 143.55 125.7) (xy 141.55 124.75) (xy 138.6 124.75) (xy 138.3 123.95) (xy 136.9 123.95)
+				(xy 136.9 125.65) (xy 140.75 125.65) (xy 142.2 126.85)
 			)
 		)
@@
 		(layer "F.Cu")
 		(hatch edge 0.5)
-		(priority 10)
+		(priority 7)
 		(connect_pads yes
 			(clearance 0.127)
@@
 			(thermal_bridge_width 0.5)
 			(smoothing fillet)
-			(radius 0.5)
+			(radius 1)
 		)
 		(polygon
 			(pts
-				(xy 143.55 126.85) (xy 143.55 125.7) (xy 141.55 124.75) (xy 138.6 124.75) (xy 138.3 123.95) (xy 136.9 123.95)
-				(xy 136.9 125.65) (xy 140.75 125.65) (xy 142.2 126.85)
+				(xy 116.95 130.65) (xy 116.95 126.2) (xy 119.25 126.2) (xy 120.25 128.1) (xy 120.24 128.9) (xy 119.25 130.65)
 			)
 		)
 	)
 	(zone
-		(net 14)
-		(net_name "+3V3")
+		(net 57)
+		(net_name "~{NMI}")
 		(layer "F.Cu")
-		(hatch edge 0.5)
-		(priority 7)
+		(name "$teardrop_padvia$")
+		(hatch none 0.1)
+		(priority 30000)
+		(attr
+			(teardrop
+				(type padvia)
+			)
+		)
 		(connect_pads yes
-			(clearance 0.127)
+			(clearance 0)
 		)
-		(min_thickness 0.25)
+		(min_thickness 0.0254)
 		(filled_areas_thickness no)
 		(fill yes
 			(thermal_gap 0.5)
 			(thermal_bridge_width 0.5)
-			(smoothing fillet)
-			(radius 1)
+			(island_removal_mode 1)
+			(island_area_min 10)
 		)
 		(polygon
 			(pts
-				(xy 116.95 130.65) (xy 116.95 126.2) (xy 119.25 126.2) (xy 120.25 128.1) (xy 120.24 128.9) (xy 119.25 130.65)
+				(xy 125.078171 99.758748) (xy 125.147934 99.784502) (xy 125.200463 99.814001) (xy 125.268757 99.881548)
+				(xy 125.309033 99.947495) (xy 125.372209 100.045521) (xy 125.420603 100.097024) (xy 125.488004 100.149441)
+				(xy 125.655633 99.900285) (xy 125.596148 99.605764) (xy 125.444131 99.64281) (xy 125.370739 99.661579)
+				(xy 125.302005 99.669978) (xy 125.221913 99.663351) (xy 125.11445 99.637041)
 			)
 		)
@@
 	)
 	(zone
+		(net 22)
+		(net_name "Net-(C59-Pad2)")
+		(layer "B.Cu")
+		(hatch edge 0.5)
+		(priority 1)
+		(connect_pads yes
+			(clearance 0.127)
+		)
+		(min_thickness 0.25)
+		(filled_areas_thickness no)
+		(fill yes
+			(thermal_gap 0.5)
+			(thermal_bridge_width 0.5)
+		)
+		(polygon
+			(pts
+				(xy 141.8 85.82) (xy 141.8 81.8) (xy 141.337154 81.8) (xy 140.053641 83.671644) (xy 140.053641 83.894178)
+				(xy 141.374308 85.82)
+			)
+		)
+	)
+	(zone
 		(net 57)
 		(net_name "~{NMI}")
@@
 	)
 	(zone
-		(net 22)
-		(net_name "Net-(C59-Pad2)")
-		(layer "B.Cu")
-		(hatch edge 0.5)
-		(priority 1)
-		(connect_pads yes
-			(clearance 0.127)
-		)
-		(min_thickness 0.25)
-		(filled_areas_thickness no)
-		(fill yes
-			(thermal_gap 0.5)
-			(thermal_bridge_width 0.5)
-		)
-		(polygon
-			(pts
-				(xy 141.8 85.82) (xy 141.8 81.8) (xy 141.337154 81.8) (xy 140.053641 83.671644) (xy 140.053641 83.894178)
-				(xy 141.374308 85.82)
-			)
-		)
-	)
-	(zone
 		(net 14)
 		(net_name "+3V3")
@@
 	)
 	(zone
-		(net 57)
-		(net_name "~{NMI}")
-		(layer "B.Cu")
-		(name "$teardrop_padvia$")
-		(hatch none 0.1)
-		(priority 30001)
-		(attr
-			(teardrop
-				(type padvia)
-			)
-		)
-		(connect_pads yes
-			(clearance 0)
-		)
-		(min_thickness 0.0254)
-		(filled_areas_thickness no)
-		(fill yes
-			(thermal_gap 0.5)
-			(thermal_bridge_width 0.5)
-			(island_removal_mode 1)
-			(island_area_min 10)
-		)
-		(polygon
-			(pts
-				(xy 126.029961 99.434911) (xy 125.954414 99.503267) (xy 125.891406 99.544224) (xy 125.791553 99.574989)
-				(xy 125.732639 99.583687) (xy 125.596148 99.605764) (xy 125.653968 99.900707) (xy 125.948911 99.958527)
-				(xy 125.970987 99.822037) (xy 125.983467 99.743114) (xy 126.004492 99.675829) (xy 126.045959 99.607318)
-				(xy 126.119764 99.524714)
-			)
-		)
-	)
-	(zone
 		(net 14)
 		(net_name "+3V3")
@@
 			)
 		)
+	)
+	(zone
+		(net 57)
+		(net_name "~{NMI}")
+		(layer "B.Cu")
+		(name "$teardrop_padvia$")
+		(hatch none 0.1)
+		(priority 30001)
+		(attr
+			(teardrop
+				(type padvia)
+			)
+		)
+		(connect_pads yes
+			(clearance 0)
+		)
+		(min_thickness 0.0254)
+		(filled_areas_thickness no)
+		(fill yes
+			(thermal_gap 0.5)
+			(thermal_bridge_width 0.5)
+			(island_removal_mode 1)
+			(island_area_min 10)
+		)
+		(polygon
+			(pts
+				(xy 126.029961 99.434911) (xy 125.954414 99.503267) (xy 125.891406 99.544224) (xy 125.791553 99.574989)
+				(xy 125.732639 99.583687) (xy 125.596148 99.605764) (xy 125.653968 99.900707) (xy 125.948911 99.958527)
+				(xy 125.970987 99.822037) (xy 125.983467 99.743114) (xy 126.004492 99.675829) (xy 126.045959 99.607318)
+				(xy 126.119764 99.524714)
+			)
+		)
